File: poket.kicad_sch (KiCad schematic)
At the start: 86 parts, among them J1 USB-C, J2 microSD, J3 3.5mm_TRS, J4 OLED-SSD1306, J5 BATT-JST, J6 DEBUG-UART, Q1 DMG2301L, SW1 EC11E-Switch, SW2 PREV, SW3 PLAY, SW4 NEXT, SW5 BOOT, SW6 RESET, SW7 PWR, U1 ESP32-S3-WROOM-1-N16R8, U2 MCP73831-2-OT, U3 AP2112K-3.3, U4 PCM5102A, U5 PAM8908, U6 BQ27441-G1, U7 USBLC6-2SC6

Commit message: Rev B: swap to ESP32-WROOM-32E-R2 so Bluetooth audio actually works
The ESP32-S3 has Bluetooth LE only - no BR/EDR - so A2DP source, the whole
point of "sends to Bluetooth headphones", could never have worked on it.
ESP-IDF's own soc_caps.h is explicit: esp32 defines SOC_BT_CLASSIC_SUPPORTED,
esp32s3 does not, and CONFIG_BT_CLASSIC_ENABLED is not even a symbol there.

New MCU: ESP32-WROOM-32E-N16R2 (ESP32-D0WDR2-V3, Classic BT + BLE, 16 MB
flash, 2 MB PSRAM in the chip package so GPIO16/17 stay free unlike a WROVER).

Knock-on changes, all verified against datasheets:
- CP2102N-A02-GQFN24 USB-UART bridge; this part has no native USB.
  VBUS sense gets the datasheet's required 22.1k/47.5k divider (abs max on
  that pin is VIO+2.5 V), RSTb a 1k pull-up to VIO, and 4.7uF + 0.1uF at
  every power pin.
- Auto-reset pair wired to Espressif's DevKitC truth table: cross-coupled,
  Q_EN base=DTR emitter=RTS, Q_IO0 base=RTS emitter=DTR, so asserting both
  lines - which opening a serial port does - resets nothing.
- microSD moved from 4-bit SDIO to SPI. The classic ESP32's 4-bit slot puts
  DAT2 on GPIO12/MTDI, the flash-voltage strap; a card's pull-up there tells
  the bootloader the flash is 1.8 V and bricks the boot.
- Battery-sense divider removed: ADC1 is fully consumed by the encoder and
  the input-only buttons, ADC2 dies when Wi-Fi is up, and the BQ27441 already
  reports voltage over I2C.
- GPIO2 strap gets a pull-down; a WS2812 data pin is high-Z.

Firmware: new pin map in board.h, SD over SPI, A2DP compiled in for real
(esp_a2d_source_init is in the binary), plus the app shell, Wi-Fi AP and the
HTTP server that serves the gzipped web UI from rodata.

Schematic ERC 0 errors / 0 warnings; all 20 firmware pins checked against the
netlist export. PCB re-placed and re-routed from scratch: DRC 0 errors, 0
schematic-parity issues, every signal net routed. Three ground-pour fragments
remain untied, two of which carry a bypass cap's ground - documented, not
hidden. Enclosur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
Parts:
- removed R21, R22: 100k, Resistor_SMD:R_0603_1608Metric, symbol Device:R
- removed U1: ESP32-S3-WROOM-1-N16R8, RF_Module:ESP32-S3-WROOM-1, symbol RF_Module:ESP32-S3-WROOM-1
- added C32, C35: 4.7uF, Capacitor_SMD:C_0603_1608Metric, symbol Device:C
- added C33, C34, C36: 100nF, Capacitor_SMD:C_0603_1608Metric, symbol Device:C
- added Q2, Q3: MMBT3904, Package_TO_SOT_SMD:SOT-23, symbol Transistor_BJT:MMBT3904
- added R31, R32: 1k, Resistor_SMD:R_0603_1608Metric, symbol Device:R
- added R33, R36, R37, R38: 10k, Resistor_SMD:R_0603_1608Metric, symbol Device:R
- added R34: 22.1k, Resistor_SMD:R_0603_1608Metric, symbol Device:R
- added R35: 47.5k, Resistor_SMD:R_0603_1608Metric, symbol Device:R
- added U1: ESP32-WROOM-32E-R2, RF_Module:ESP32-WROOM-32E, symbol RF_Module:ESP32-WROOM-32E-R2
- added U8: CP2102N-A02-GQFN24, Package_DFN_QFN:QFN-24-1EP_4x4mm_P0.5mm_EP2.6x2.6mm, symbol Interface_USB:CP2102N-Axx-xQFN24
Connections:
- net 3V3: now also R33.1, U1.2 (VDD)
- net AMP_EN: now also U1.26 (IO4)
- net BTN_NEXT: now also U1.5 (SENSOR_VN)
- net BTN_PLAY: now also U1.4 (SENSOR_VP)
- net BTN_PREV: now also U1.6 (IO34)
- net DAC_XSMT: now also U1.13 (IO14)
- net ENC_A: now also U1.8 (IO32)
- net ENC_B: now also U1.9 (IO33)
- net ENC_SW: now also U1.7 (IO35)
- net ESP_EN: now also Q2.3 (C), U1.3 (EN)
- net ESP_IO0: now also Q3.3 (C), U1.25 (IO0)
- net GND: now also C32.2, C33.2, C34.2, C35.2, C36.2, R35.2, R38.2, U1.[1,15,38,39] (GND), U8.18 (~{CTS}), U8.2 (GND), U8.22 (~{DSR}), U8.24 (~{DCD}), U8.25 (GND)
- net I2C_SCL: now also U1.36 (IO22)
- net I2C_SDA: now also U1.33 (IO21)
- net I2S_BCK: now also U1.11 (IO26)
- net I2S_DIN: now also U1.12 (IO27)
- net I2S_LRCK: now also U1.10 (IO25)
- net JACK_DET: now also U1.23 (IO15)
- net LED_DIN: now also R38.1, U1.24 (IO2)
- net SD_CD: now also U1.16 (IO13)
- net UART_RX: now also R33.2, U1.34 (RXD0/IO3), U8.21 (TXD)
- net UART_TX: now also R32.1, U1.35 (TXD0/IO1)
- net USB_DM: now also U8.4 (D-)
- net USB_DP: now also U8.3 (D+)
- net VBUS: now also C33.1, C35.1, R34.1, U8.7 (VREGIN)
- net FG_GPOUT: no longer names the net of U6.12 (GPOUT)
- net SD_CLK renamed SD_SCK
- net SD_SCK: now also U1.30 (IO18)
- net SD_CMD renamed SD_MOSI
- net SD_MOSI: now also U1.37 (IO23)
- net SD_D0 renamed SD_MISO
- net SD_MISO: now also U1.31 (IO19)
- net SD_D3 renamed SD_CS
- net SD_CS: now also U1.29 (IO5)
- new net CP_RSTN: R31.2, U8.9 (~{RST})
- new net CP_RXD: R32.2, U8.20 (RXD)
- new net CP_VBSENSE: R34.2, R35.1, U8.8 (VBUS)
- new net CP_VDD: C32.1, C34.1, C36.1, R31.1, U8.5 (VIO), U8.6 (VDD)
- new net Q2_BASE: Q2.1 (B), R36.2
- new net Q3_BASE: Q3.1 (B), R37.2
- new net UART_DTR: Q3.2 (E), R36.1, U8.23 (~{DTR})
- new net UART_RTS: Q2.2 (E), R37.1, U8.19 (~{RTS})
- no-connect marks 15 -> 18
